File: HARDWARE/ELECTRICAL/pov_display/pov_display.kicad_pcb (KiCad board)
At the start: 2 copper layers, 345.8 x 103.8 mm, 50 parts, among them J1 Conn_01x04_Male, J2 Conn_01x04_Male, J3 Screw_Terminal_01x02, SW1 SW_Push, U1 Pico, U2 74AHCT125, U3 DRV5033AJxLPG

Commit message: Updated schematic for correct silkscreen labels
Parts:
- moved SW1 28.0 mm to (95.0, 147.5)
- moved U2 28.0 mm to (96.2, 113.5)
- moved C1 28.0 mm to (141.4, 114.2)
- moved D41 28.0 mm to (138.4, 120.6)
- moved J1 28.0 mm to (95.7, 128.2)
- moved J3 28.0 mm to (141.4, 106.6)
- moved R1 28.0 mm to (135.2, 143.3)
- moved U1 28.0 mm to (118.1, 128.2)
- moved U3 28.0 mm to (141.2, 150.7)
- moved D21 6.15 mm to (252.8, 62.6)
- moved D25 6.15 mm to (283.3, 62.6)
- moved D26 6.15 mm to (290.9, 62.6)
- moved D27 6.15 mm to (298.5, 62.6)
- moved D28 6.15 mm to (306.1, 62.6)
- moved D29 6.15 mm to (313.7, 62.6)
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Other:
- board size 345.8 x 103.8 mm -> 345 x 107.3 mm
